File: Input_Output.kicad_sch (KiCad schematic)
At the start: 18 parts, among them J1 Conn_01x04, J13 Conn_ARM_SWD_TagConnect_TC203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, J14 Conn_01x06, J2 Conn_01x06, J3 Conn_01x02, J7 Conn_01x05, J8 USB_B_Micro, J9 Conn_ARM_SWD_TagConnect_TC203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, U32 Micro_SD_Card_Det1

Commit message: Finalize schematics as AIoT2-rev003-May1326
Parts:
- added R8: 360, Resistor_SMD:R_0402_1005Metric, symbol Device:R_Small
- C10, C9: footprint (none) -> Capacitor_SMD:C_0402_1005Metric
- J1: footprint (none) -> Connector_PinHeader_2.54mm:PinHeader_1x04_P2.54mm_Vertical
- J14, J2: footprint (none) -> Connector_PinHeader_2.54mm:PinHeader_1x06_P2.54mm_Vertical
- J3: footprint (none) -> Connector_PinHeader_2.54mm:PinHeader_1x02_P2.54mm_Vertical
- J7: footprint (none) -> Connector_PinHeader_2.54mm:PinHeader_1x05_P2.54mm_Vertical
- J8: footprint (none) -> Connector_USB:USB_Micro-B_Molex-105017-0001
- J_5V1: renamed from J_5V; footprint (none) -> TestPoint:TestPoint_Pad_D1.0mm
- J_D+1: renamed from J_D+; footprint (none) -> TestPoint:TestPoint_Pad_D1.0mm
- J_D-1: renamed from J_D-; footprint (none) -> TestPoint:TestPoint_Pad_D1.0mm
- J_GND1: renamed from J_GND; footprint (none) -> TestPoint:TestPoint_Pad_D1.0mm
- R6: footprint (none) -> Resistor_SMD:R_0402_1005Metric
- SW_User1: renamed from SW_User; footprint (none) -> Button_Switch_SMD:Panasonic_EVQPUM_EVQPUD
- U32: footprint (none) -> footprints:microSD_XKB_XKTF-015-x
- renumbered LED1 to D1
Connections:
- net GND: now also R8.2; no longer D1.1 (K)
- new net: D1.1 (K), R8.1
Other:
- title: (none) -> UCA DKAIoT2 — Input/Output
