File: Input_Output.kicad_sch (KiCad schematic)
At the start: 17 parts, among them J1 Conn_01x04, J2J14 Conn_02x06_Odd_Even, J3 Conn_01x02, J7 Conn_01x05, J8 USB_B_Micro, J9J13 Conn_ARM_SWD_TagConnect_TC203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, U32 Micro_SD_Card_Det1

Commit message: WIP: remove unneeded parts from PCB, add SPA06 and FHTC3 to schematics
Parts:
- J2J14, J3, J_5V1, J_D+1, J_D-1, J_GND1: now not fitted; now left out of the parts list
- J9J13: now not fitted
Connections:
- net I2C3_SCL renamed I2C2_SCL
- net I2C3_SDA renamed I2C2_SDA
Changed lines of the file:
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@@
 		)
 	)
-	(global_label "I2C3_SCL"
+	(global_label "I2C2_SCL"
 		(shape input)
 		(at 78.74 118.11 0)
@@
 		)
 	)
-	(global_label "I2C3_SDA"
+	(global_label "I2C2_SDA"
 		(shape bidirectional)
 		(at 78.74 115.57 0)
@@
 					(reference "C10")
 					(unit 1)
-					(variant
-						(name "Ambient")
-					)
 				)
 			)
@@
 		(body_style 1)
 		(exclude_from_sim no)
-		(in_bom yes)
-		(on_board yes)
-		(in_pos_files yes)
-		(dnp no)
+		(in_bom no)
+		(on_board no)
+		(in_pos_files no)
+		(dnp yes)
 		(fields_autoplaced yes)
 		(property "Reference" "J_GND1"
@@
 					(variant
 						(name "Ambient")
+						(dnp no)
+						(in_bom yes)
+						(on_board yes)
+						(in_pos_files yes)
 					)
 				)
@@
 		(body_style 1)
 		(exclude_from_sim no)
-		(in_bom yes)
-		(on_board yes)
-		(in_pos_files yes)
-		(dnp no)
+		(in_bom no)
+		(on_board no)
+		(in_pos_files no)
+		(dnp yes)
 		(fields_autoplaced yes)
 		(property "Reference" "J_D+1"
@@
 					(variant
 						(name "Ambient")
+						(dnp no)
+						(in_bom yes)
+						(on_board yes)
+						(in_pos_files yes)
 					)
 				)
@@
 					(reference "R6")
 					(unit 1)
-					(variant
-						(name "Ambient")
-					)
 				)
 			)
@@
 					(reference "D1")
 					(unit 1)
-					(variant
-						(name "Ambient")
-					)
 				)
 			)
@@
 		(body_style 1)
 		(exclude_from_sim no)
-		(in_bom yes)
-		(on_board yes)
-		(in_pos_files yes)
-		(dnp no)
+		(in_bom no)
+		(on_board no)
+		(in_pos_files no)
+		(dnp yes)
 		(fields_autoplaced yes)
 		(property "Reference" "J3"
@@
 					(variant
 						(name "Ambient")
-						(dnp yes)
+						(in_bom yes)
+						(on_board yes)
+						(in_pos_files yes)
 					)
 				)
@@
 					(reference "U32")
 					(unit 1)
-					(variant
-						(name "Ambient")
-					)
 				)
 			)
@@
 					(reference "R8")
 					(unit 1)
-					(variant
-						(name "Ambient")
-					)
 				)
 			)
@@
 					(reference "C9")
 					(unit 1)
-					(variant
-						(name "Ambient")
-					)
 				)
 			)
@@
 		(exclude_from_sim no)
 		(in_bom no)
-		(on_board yes)
-		(in_pos_files yes)
-		(dnp no)
+		(on_board no)
+		(in_pos_files no)
+		(dnp yes)
 		(property "Reference" "J9J13"
 			(at 146.05 82.5499 0)
@@
 					(variant
 						(name "Ambient")
+						(dnp no)
+						(on_board yes)
+						(in_pos_files yes)
 					)
 				)
@@
 		(body_style 1)
 		(exclude_from_sim no)
-		(in_bom yes)
-		(on_board yes)
-		(in_pos_files yes)
-		(dnp no)
+		(in_bom no)
+		(on_board no)
+		(in_pos_files no)
+		(dnp yes)
 		(property "Reference" "J2J14"
 			(at 73.406 128.524 0)
@@
 		(body_style 1)
 		(exclude_from_sim no)
-		(in_bom yes)
-		(on_board yes)
-		(in_pos_files yes)
-		(dnp no)
+		(in_bom no)
+		(on_board no)
+		(in_pos_files no)
+		(dnp yes)
 		(fields_autoplaced yes)
 		(property "Reference" "J_D-1"
@@
 					(variant
 						(name "Ambient")
+						(dnp no)
+						(in_bom yes)
+						(on_board yes)
+						(in_pos_files yes)
 					)
 				)
@@
 		(body_style 1)
 		(exclude_from_sim no)
-		(in_bom yes)
-		(on_board yes)
-		(in_pos_files yes)
-		(dnp no)
+		(in_bom no)
+		(on_board no)
+		(in_pos_files no)
+		(dnp yes)
 		(fields_autoplaced yes)
 		(property "Reference" "J_5V1"
@@
 					(variant
 						(name "Ambient")
+						(dnp no)
+						(in_bom yes)
+						(on_board yes)
+						(in_pos_files yes)
 					)
 				)
@@
 					(reference "J8")
 					(unit 1)
-					(variant
-						(name "Ambient")
-					)
 				)
 			)
@@
 					(reference "SW_User1")
 					(unit 1)
-					(variant
-						(name "Ambient")
-					)
 				)
 			)

Commit message: WIP: import ambient-pcb-lifepo4protection and ambient-pcb-audiopower schematics
Connections:
- net VDD_1V8 renamed +1V8
- net V_PERIPH_3V renamed +3V0_PERIPH

Commit message: WIP: BOM
Parts:
- removed D1: LED_0603_Blue, PCM_LED_SMD_AKL:LED_0603_1608Metric, symbol PCM_LED_AKL:LED_0603_Blue
- added D1: LED_0805_Green, PCM_LED_SMD_AKL:LED_0805_2012Metric, symbol PCM_LED_AKL:LED_0805_Green
- C10, C9: LCSC (none) -> C1525
- J1: footprint Connector_PinHeader_2.54mm:PinHeader_1x04_P2.54mm_Vertical -> Connector_JST:JST_XH_B4B-XH-A_1x04_P2.50mm_Vertical; LCSC (none) -> C37815; now not fitted; now left out of the parts list
- J2J14: LCSC (none) -> C36191
- J3: footprint Connector_PinHeader_2.54mm:PinHeader_1x02_P2.54mm_Vertical -> Connector_JST:JST_XH_B2B-XH-A_1x02_P2.50mm_Vertical; LCSC (none) -> C20079
- J7: footprint Connector_PinHeader_2.54mm:PinHeader_1x05_P2.54mm_Vertical -> Connector_JST:JST_XH_B5B-XH-A_1x05_P2.50mm_Vertical; LCSC (none) -> C2318; now not fitted
- J8: footprint Connector_USB:USB_Micro-B_Molex-105017-0001 -> Connector_USB:USB_Micro-B_Amphenol_10118194-0001LF_Horizontal; LCSC (none) -> C132563
- R6: LCSC (none) -> C25900
- R8: value 360 -> 1k; LCSC (none) -> C11702
- SW_User1: LCSC (none) -> C223812
- U32: LCSC (none) -> C22383473
Connections:
- net +3V0_PERIPH: no longer U32.4 (VDD)
- net LED: now also D1.2 (A)
- net at R8.1: now also D1.1 (K)
- new net +3V0_SD: U32.4 (VDD)

Commit message: Finish routing + silkscreen placement
Parts:
- SW_User1: FT Rotation Offset (none) -> 180
- U32: FT Position Offset (none) -> 0.127,0.0
Changed lines of the file:
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@@
+			)
+		)
+		(property "FT Position Offset" "0.127,0.0"
+			(at 86.36 59.69 0)
+			(hide yes)
+			(show_name no)
+			(do_not_autoplace no)
+			(effects
+				(font
+					(size 1.27 1.27)
+				)
 			)
 		)
@@
 			(at 59.69 167.64 0)
 			(hide yes)
+			(show_name no)
+			(do_not_autoplace no)
+			(effects
+				(font
+					(size 1.27 1.27)
+				)
+			)
+		)
+		(property "FT Rotation Offset" "180"
+			(at 59.69 167.64 0)
+			(hide yes)

Commit message: JLCPCB offsets and small fixes
Parts:
- U32: FT Position Offset 0.127,0.0 -> -0.0635,0.127
Changed lines of the file:
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@@
 			)
 		)
-		(property "FT Position Offset" "0.127,0.0"
+		(property "FT Position Offset" "-0.0635,0.127"
 			(at 86.36 59.69 0)
 			(hide yes)
