File: LoRa.kicad_sch (KiCad schematic)
At the start: 17 parts, among them J10 Conn_01x03, J6 Conn_01x03, U1 NCV8170AXV300T2G, U2 Quectel_L96, U5 E22-900M22S

Commit message: Continue filling schematics
Other:
- company: (none) -> //piernov
Changed lines of the file:
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@@
 	(generator_version "10.0")
 	(paper "A4")
+	(title_block
+		(date "2026-05-27")
+		(rev "v0.1")
+		(company "//piernov")
+	)
 	(text_box "GNSS receiver"
 		(exclude_from_sim no)

Commit message: Finalize schematics as AIoT2-rev003-May1326
Parts:
- removed J10, J6: Conn_01x03, symbol Connector_Generic:Conn_01x03
- added C20: 100nF, Capacitor_SMD:C_0402_1005Metric, symbol Device:C_Small
- added J10, J6: Conn_Coaxial, Connector_Coaxial:U.FL_Hirose_U.FL-R-SMT-1_Vertical, symbol Connector:Conn_Coaxial
- C1, C2: footprint (none) -> Capacitor_SMD:C_0402_1005Metric
- J_GPS_EN1: renamed from J_GPS_EN; footprint (none) -> TestPoint:TestPoint_Pad_D1.0mm
- J_RX1: renamed from J_RX; footprint (none) -> TestPoint:TestPoint_Pad_D1.0mm
- J_TX1: renamed from J_TX; footprint (none) -> TestPoint:TestPoint_Pad_D1.0mm
- R1, R2, R26, R27, R3, R4, R5: footprint (none) -> Resistor_SMD:R_0402_1005Metric
- U5: footprint RF_Module:E22-400M22S -> footprints:E22-400M22S
Connections:
- net E22_ANT: now also J10.1 (In), J6.1 (In)
- net GND: now also C20.2, J10.2 (Ext), J6.2 (Ext)
- net V_PERIPH_3V: now also C20.1
- no-connect marks 5 -> 6
Other:
- title: (none) -> UCA DKAIoT2 — Wireless
