File: LoRa.kicad_sch (KiCad schematic)
At the start: 26 parts, among them J10 Conn_Coaxial, J20 Conn_01x01, J21 Conn_01x01, J22 Conn_01x01, J23 Conn_01x01, J24 Conn_01x01, J25 Conn_01x01, J26 Conn_01x01, J6 Conn_Coaxial, U1 NCV8170AXV300T2G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

Commit message: v0.2: fix Ebyte E22-900M22S pinout
Connections:
- net GND: now also U5.10 (GND)
- net V_PERIPH_3V: no longer U5.10 (VCC)
Changed lines of the file:
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@@
 	(title_block
 		(title "UCA DKAIoT2 — Wireless")
-		(date "2026-06-05")
-		(rev "v0.1")
+		(date "2026-06-14")
+		(rev "v0.2")
 		(company "//piernov")
 	)
