File: Power.kicad_sch (KiCad schematic)
At the start: 33 parts, among them J11 Conn_01x02, J12 Conn_01x02, J4 Conn_01x02, J5 Conn_01x02, U10 NCV8170AXV300T2G, U26 NCV8170AXV180T2G, U3 Conn_01x04, U3 MCP73831-2-OT, U33 NCV8170AXV300T2G

Commit message: Continue filling schematics
Parts:
- added C16, C42: 470µF, symbol Device:C_Polarized_Small
- added C33, C35: 100nF, symbol Device:C_Small
- added C34, C36: 10nF, symbol Device:C_Small
- added R18, R20: 330, symbol Device:R_Small
- added R19, R21: 1k, symbol Device:R_Small
- added R22, R23: 0, symbol Device:R_Small
- added R39, R40: 4.7k, symbol Device:R_Small
- added R41, R42, R43, R44: 10k, symbol Device:R_Small
- added U12, U15: R5478N101CD, Package_TO_SOT_SMD:SOT-23-6, symbol Nisshinbo_R5478N:R5478N101CD
- added U13, U14, U16, U17: FDV301N, PCM_Package_TO_SOT_SMD_AKL:SOT-23, symbol PCM_Transistor_MOSFET_AKL:FDV301N
- added U28, U30, U31: BSS138L, PCM_Package_TO_SOT_SMD_AKL:SOT-23, symbol PCM_Transistor_MOSFET_AKL:BSS138L
Connections:
- net +BATT1_IN is gone; now on net +BATT: J11.2 (Pin_2), U3.1 (Pin_1)
- net +BATT2_IN is gone; now on net +BATT: J12.2 (Pin_2), U3.2 (Pin_2)
- net +BATT: now also C33.1, C35.1, R18.1, R20.1
- net -BATT1_IN: now also R19.2, R22.2, U14.2 (S)
- net -BATT2_IN: now also R21.2, R23.2, U17.2 (S)
- net GND: now also C16.2, C33.2, C34.2, C35.2, C36.2, C42.2, R22.1, R23.1, U12.6 (VSS), U13.2 (S), U15.6 (VSS), U16.2 (S)
- net VDD_1V8: now also R39.1, R42.1, R44.1, U28.1 (G), U30.1 (G), U31.1 (G)
- net V_PERIPH_3V: now also C16.1, C42.1, R40.1, R41.1, R43.1
- new net: U12.3 (COUT), U14.1 (G)
- new net: U13.3 (D), U14.3 (D)
- new net: C34.1, R18.2, U12.5 (VDD)
- new net: R21.1, U15.2 (V-)
- new net: U12.1 (DOUT), U13.1 (G)
- new net: R19.1, U12.2 (V-)
- new net: U15.3 (COUT), U17.1 (G)
- new net: U16.3 (D), U17.3 (D)
- new net: U15.1 (DOUT), U16.1 (G)
- new net: C36.1, R20.2, U15.5 (VDD)
- new net I2C1_SCL: R43.2, U31.3 (D)
- new net I2C1_SDA: R41.2, U30.3 (D)
- new net ICM_INT: R40.2, U28.3 (D)
- new net ICM_INT_1V8: R39.2, U28.2 (S)
- new net SCL_1V8: R44.2, U31.2 (S)
- new net SDA_1V8: R42.2, U30.2 (S)
Other:
- company: (none) -> //piernov
- moved on the sheet: C26, C27, C54, C55, C56, C57, D2, D3, D6, J11, J12, J4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

Commit message: Finalize schematics as AIoT2-rev003-May1326
Parts:
- C16, C42: footprint (none) -> Capacitor_Tantalum_SMD:CP_EIA-7343-15_Kemet-W
- C26, C27, C28, C29, C30, C31, C33, C34, C35, C36, C51, C54, C55, C56, C57: footprint (none) -> Capacitor_SMD:C_0402_1005Metric
- J11, J12, J4, J5: footprint (none) -> Connector_PinHeader_2.54mm:PinHeader_1x02_P2.54mm_Vertical
- J_3V1: renamed from J_3V; footprint (none) -> TestPoint:TestPoint_Pad_D1.0mm
- J_PERIPH_3V1: renamed from J_PERIPH_3V; footprint (none) -> TestPoint:TestPoint_Pad_D1.0mm
- J_PERIPH_CTRL1: renamed from J_PERIPH_CTRL; footprint (none) -> TestPoint:TestPoint_Pad_D1.0mm
- R15, R16, R18, R19, R20, R21, R22, R23, R39, R41, R42, R43, R44, R54, R55, R56: footprint (none) -> Resistor_SMD:R_0402_1005Metric
- R38: renamed from R40; footprint (none) -> Resistor_SMD:R_0402_1005Metric
- U26: value NCV8170AXV180T2G -> NCV8170BXV180T2G
- U3: footprint (none) -> footprints:BAT-TH_BH-18650-A1BJ034
- renumbered U3 to U9
Connections:
- net Vin: now also C28.1, D4.1 (K), D5.1 (K), U10.1 (IN), U10.6 (EN)
- net CHRG_PWR_IN: no longer names the net of C26.1, D2.1 (K), D3.1 (K), U9.4 (V_{DD})
Other:
- title: (none) -> UCA DKAIoT2 — Power
- moved on the sheet: C26, C33, C34, C35, C36, R18, R19, R20, R21, R22, R23, U12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
