File: Power.kicad_sch (KiCad schematic)
At the start: 60 parts, among them J11 Conn_01x02, J12 Conn_01x02, J4 Conn_01x02, J5 Conn_01x02, U10 NCV8170AXV300T2G, U12 R5478N101CD, U13 FDV301N, U14 FDV301N, U15 R5478N101CD, U16 FDV301N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

Commit message: schematics: add some DNP for Ambient variant
Parts:
- J4: footprint Connector_PinHeader_2.54mm:PinHeader_1x02_P2.54mm_Vertical -> Connector_PinSocket_2.54mm:PinSocket_1x02_P2.54mm_Vertical
Changed lines of the file:
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@@
 			)
 		)
-		(property "Footprint" "Connector_PinHeader_2.54mm:PinHeader_1x02_P2.54mm_Vertical"
+		(property "Footprint" "Connector_PinSocket_2.54mm:PinSocket_1x02_P2.54mm_Vertical"
 			(at 148.59 93.98 0)
 			(hide yes)
