File: Sensors.kicad_sch (KiCad schematic)
At the start: 27 parts, among them U11 DRV5023AJxLPG, U18 LTR-303ALS-01, U21 HP203B, U22 SPH0645LM4H, U29 SGP30, U7 BME280

Commit message: WIP: remove unneeded parts from PCB, add SPA06 and FHTC3 to schematics
Parts:
- added C58, C59: 100nF, Capacitor_SMD:C_0402_1005Metric, symbol Device:C_Small
- added R57: 0, Resistor_SMD:R_0402_1005Metric, symbol Device:R_Small
- added U23: SPA06-003, Package_LGA:Bosch_LGA-8_2x2.5mm_P0.65mm_ClockwisePinNumbering, symbol Sensor_Pressure:BMP280
- added U25: FHTC3, Package_DFN_QFN:DFN-6-1EP_2x2mm_P0.5mm_EP0.7x1.6mm, symbol Sensor_Humidity:GXHTC3
- C17, C23, C24, C32, C37, C39, C46, C52, C53, R10, R12, R17, R29, R30, R31, R34, R47, R49, RN1, U11, U18, U21, U22, U29, U7: now not fitted; now left out of the parts list
- R46, R48: now left out of the parts list
Connections:
- net GND: now also C58.2, C59.2, R57.2, U23.1 (GND), U23.7 (GND), U25.6 (GND), U25.7 (EPAD)
- net I2C1_SCL: now also U23.4 (SCK), U25.3 (SCL)
- net I2C1_SDA: now also U23.3 (SDI), U25.4 (SDA)
- net INT_ACC_3: now also R57.1, U23.5 (SDO)
- net V_PERIPH_3V: now also C58.1, C59.1, U23.6 (VDDIO), U23.8 (VDD), U25.1 (VDD)
- no-connect marks 4 -> 5

Commit message: WIP: import ambient-pcb-lifepo4protection and ambient-pcb-audiopower schematics
Parts:
- C17, C23, C24, C32, C37, C39, C46, C52, C53: now in the parts list
Connections:
- net VDD_1V8 renamed +1V8
- net V_PERIPH_3V renamed +3V0_PERIPH

Commit message: WIP: BOM
Parts:
- C17, C23, C24, C32, C46, C52, C53: LCSC (none) -> C1525; now left out of the parts list
- C37: LCSC (none) -> C52923; now left out of the parts list
- C39: LCSC (none) -> C23733; now left out of the parts list
- C58, C59: LCSC (none) -> C1525
- R10, R31: LCSC (none) -> C26083
- R12: LCSC (none) -> C310212
- R17: LCSC (none) -> C25900
- R30, R34, R46, R47, R48, R49: LCSC (none) -> C17168
- R57: value 0 -> 47k; LCSC (none) -> C25792
- RN1: LCSC (none) -> C1952
- U11: LCSC (none) -> C1497675
- U18: LCSC (none) -> C364577
- U21: LCSC (none) -> C138665
- U22: LCSC (none) -> C19272537
- U29: LCSC (none) -> C514454
- U7: LCSC (none) -> C92489

Commit message: Finish routing + silkscreen placement
Parts:
- U25: FT Rotation Offset (none) -> -90
Changed lines of the file:
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@@
+			)
+		)
+		(property "FT Rotation Offset" "-90"
+			(at 207.01 134.62 0)
+			(hide yes)
+			(show_name no)
+			(do_not_autoplace no)
+			(effects
+				(font
+					(size 1.27 1.27)
+				)
 			)
 		)

Commit message: JLCPCB offsets and small fixes
Parts:
- U23: FT Rotation Offset (none) -> -90
Changed lines of the file:
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@@
+			)
+		)
+		(property "FT Rotation Offset" "-90"
+			(at 262.89 43.18 0)
+			(hide yes)
+			(show_name no)
+			(do_not_autoplace no)
+			(effects
+				(font
+					(size 1.27 1.27)
+				)
 			)
 		)
