File: Sensors_IMU.kicad_sch (KiCad schematic)
At the start: 19 parts, among them U20 KXTJ3-1057, U24 KX023-1025, U4 ICM-20948, U6 LSM303AH

Commit message: Continue filling schematics
Other:
- company: (none) -> //piernov
Changed lines of the file:
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@@
 	(generator_version "10.0")
 	(paper "A4")
+	(title_block
+		(date "2026-05-27")
+		(rev "v0.1")
+		(company "//piernov")
+	)
 	(text_box "TDK ICM-20948: 3-axis accelerometer, 3-axis gyroscope, 3-axis magnetometer"
 		(exclude_from_sim no)

Commit message: Finalize schematics as AIoT2-rev003-May1326
Parts:
- C21, C22, C38, C40, C41, C47, C48, C50: footprint (none) -> Capacitor_SMD:C_0402_1005Metric
- C49: renamed from C39; footprint (none) -> Capacitor_SMD:C_0402_1005Metric
- R35, R36, R50, R51, R52, R53: footprint (none) -> Resistor_SMD:R_0402_1005Metric
- renumbered U4 to U19
Other:
- title: (none) -> UCA DKAIoT2 — Sensors Motion
Changed lines of the file:
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@@
 	(paper "A4")
 	(title_block
-		(date "2026-05-27")
+		(title "UCA DKAIoT2 — Sensors Motion")
+		(date "2026-05-28")
 		(rev "v0.1")
 		(company "//piernov")
@@
 	)
 	(global_label "ICM_INT_1V8"
-		(shape input)
+		(shape output)
 		(at 54.61 57.15 180)
 		(fields_autoplaced yes)
@@
 	)
 	(global_label "INT_ACC_2"
-		(shape input)
+		(shape output)
 		(at 85.09 113.03 0)
 		(fields_autoplaced yes)
@@
 	)
 	(global_label "INT_ACC_1"
-		(shape input)
+		(shape output)
 		(at 85.09 110.49 0)
 		(fields_autoplaced yes)
@@
 	)
 	(global_label "INT_ACC_3"
-		(shape input)
+		(shape output)
 		(at 85.09 115.57 0)
 		(fields_autoplaced yes)
@@
 	)
 	(global_label "I2C1_SDA"
-		(shape input)
+		(shape bidirectional)
 		(at 41.91 113.03 180)
 		(fields_autoplaced yes)
@@
 		)
 		(property "Intersheetrefs" "${INTERSHEET_REFS}"
-			(at 30.0953 113.03 0)
+			(at 28.984 113.03 0)
 			(hide yes)
 			(show_name no)
@@
 	)
 	(global_label "I2C1_SDA"
-		(shape input)
+		(shape bidirectional)
 		(at 148.59 45.72 180)
 		(fields_autoplaced yes)
@@
 		)
 		(property "Intersheetrefs" "${INTERSHEET_REFS}"
-			(at 136.7753 45.72 0)
+			(at 135.664 45.72 0)
 			(hide yes)
 			(show_name no)
@@
 	)
 	(global_label "INT_ACC_2"
-		(shape input)
+		(shape output)
 		(at 176.53 48.26 0)
 		(fields_autoplaced yes)
@@
 	)
 	(global_label "I2C1_SDA"
-		(shape input)
+		(shape bidirectional)
 		(at 161.29 113.03 0)
 		(fields_autoplaced yes)
@@
 		)
 		(property "Intersheetrefs" "${INTERSHEET_REFS}"
-			(at 173.1047 113.03 0)
+			(at 174.216 113.03 0)
 			(hide yes)
 			(show_name no)
@@
 	)
 	(global_label "SDA_1V8"
-		(shape input)
+		(shape bidirectional)
 		(at 54.61 44.45 180)
 		(fields_autoplaced yes)
@@
 		)
 		(property "Intersheetrefs" "${INTERSHEET_REFS}"
-			(at 43.5815 44.45 0)
+			(at 42.4702 44.45 0)
 			(hide yes)
 			(show_name no)
@@
 	)
 	(global_label "INT_ACC_1"
-		(shape input)
+		(shape output)
 		(at 176.53 45.72 0)
 		(fields_autoplaced yes)
@@
 	)
 	(global_label "INT_ACC_1"
-		(shape input)
+		(shape output)
 		(at 161.29 107.95 0)
 		(fields_autoplaced yes)
@@
 			)
 		)
-		(property "Footprint" ""
+		(property "Footprint" "Resistor_SMD:R_0402_1005Metric"
 			(at 176.53 120.65 0)
 			(hide yes)
@@
 			)
 		)
-		(property "Footprint" ""
+		(property "Footprint" "Resistor_SMD:R_0402_1005Metric"
 			(at 38.1 46.99 0)
 			(hide yes)
@@
 			)
 		)
-		(property "Footprint" ""
+		(property "Footprint" "Capacitor_SMD:C_0402_1005Metric"
 			(at 124.46 48.26 0)
 			(hide yes)
@@
 			)
 		)
-		(property "Footprint" ""
+		(property "Footprint" "Capacitor_SMD:C_0402_1005Metric"
 			(at 135.89 113.03 0)
 			(hide yes)
@@
 			)
 		)
-		(property "Footprint" ""
+		(property "Footprint" "Capacitor_SMD:C_0402_1005Metric"
 			(at 194.31 46.99 0)
 			(hide yes)
@@
 			)
 		)
-		(property "Footprint" ""
+		(property "Footprint" "Resistor_SMD:R_0402_1005Metric"
 			(at 133.35 53.34 0)
 			(hide yes)
@@
 			)
 		)
-		(property "Footprint" ""
+		(property "Footprint" "Capacitor_SMD:C_0402_1005Metric"
 			(at 85.09 59.69 0)
 			(hide yes)
@@
 			)
 		)
-		(property "Footprint" ""
+		(property "Footprint" "Capacitor_SMD:C_0402_1005Metric"
 			(at 85.09 125.73 0)
 			(hide yes)
@@
 		(dnp no)
 		(fields_autoplaced yes)
-		(property "Reference" "U4"
+		(property "Reference" "U19"
 			(at 71.9933 67.31 0)
 			(show_name no)
@@
 			(project "uca-dkaiot2-kicad"
 				(path "/13b7de53-ecff-4b32-b513-b5b471d022a3/177e1d79-4046-4c8a-85e5-b39397a261aa"
-					(reference "U4")
+					(reference "U19")
 					(unit 1)
 				)
@@
 			)
 		)
-		(property "Footprint" ""
+		(property "Footprint" "Resistor_SMD:R_0402_1005Metric"
 			(at 176.53 110.49 0)
 			(hide yes)
@@
 			)
 		)
-		(property "Footprint" ""
+		(property "Footprint" "Resistor_SMD:R_0402_1005Metric"
 			(at 133.35 43.18 0)
 			(hide yes)
@@
 		(in_pos_files yes)
 		(dnp no)
-		(property "Reference" "C39"
+		(property "Reference" "C49"
 			(at 19.558 41.91 0)
 			(show_name no)
@@
 			)
 		)
-		(property "Footprint" ""
+		(property "Footprint" "Capacitor_SMD:C_0402_1005Metric"
 			(at 29.21 43.18 0)
 			(hide yes)
@@
 			(project "uca-dkaiot2-kicad"
 				(path "/13b7de53-ecff-4b32-b513-b5b471d022a3/177e1d79-4046-4c8a-85e5-b39397a261aa"
-					(reference "C39")
+					(reference "C49")
 					(unit 1)
 				)
@@
 			)
 		)
-		(property "Footprint" ""
+		(property "Footprint" "Capacitor_SMD:C_0402_1005Metric"
 			(at 95.25 46.99 0)
 			(hide yes)
@@
 			)
 		)
-		(property "Footprint" ""
+		(property "Footprint" "Capacitor_SMD:C_0402_1005Metric"
 			(at 184.15 114.3 0)
 			(hide yes)
@@
 			)
 		)
-		(property "Footprint" ""
+		(property "Footprint" "Resistor_SMD:R_0402_1005Metric"
 			(at 38.1 36.83 0)
 			(hide yes)
@@
 			)
 		)
-		(property "Footprint" ""
+		(property "Footprint" "Capacitor_SMD:C_0402_1005Metric"
 			(at 29.21 120.65 0)
 			(hide yes)
