File: Sensors_IMU.kicad_sch (KiCad schematic)
At the start: 19 parts, among them U19 ICM-20948, U20 KXTJ3-1057, U24 KX023-1025, U6 LSM303AH

Commit message: schematics: add some DNP for Ambient variant
Connections:
- new net: U24.10 (NC), U24.15 (NC), U24.16 (NC), U24.2 (NC), U24.3 (NC)
Changed lines of the file:
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@@
 		(pin "1"
+		)
+		(pin "2"
+		)
+		(pin "3"
+		)
+		(pin "16"
+		)
+		(pin "10"
+		)
+		(pin "15"
 		)
 		(instances
