File: uca-dkaiot2-kicad.kicad_pcb (KiCad board)
At the start: 4 copper layers, 156.3 x 77.5 mm, 183 parts, among them J1 Conn_01x04, J10 Conn_Coaxial, J11 Conn_01x02, J12 Conn_01x02, J20 Conn_01x01, J21 Conn_01x01, J22 Conn_01x01, J23 Conn_01x01, J24 Conn_01x01, J25 Conn_01x01, J26 Conn_01x01, J2J14 Conn_02x06_Odd_Even, J3 Conn_01x02, J4 Conn_01x02, J5 Conn_01x02, J6 Conn_Coaxial, J7 Conn_01x05, J8 USB_B_Micro, J9J13 Conn_ARM_SWD_TagConnect_TC203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, U1 NCV8170AXV300T2G, U10 NCV8170AXV300T2G, U11 DRV5023AJxLPG, U12 R5478N101CD, U13 FDV301N, U14 FDV301N, U15 R5478N101CD, U16 FDV301N, U17 FDV301N, U18 LTR-303ALS-01, U19 ICM-20948, U2 Quectel_L96, U20 KXTJ3-1057, U21 HP203B, U22 SPH0645LM4H, U24 KX023-1025, U26 NCV8170BXV180T2G, U28 BSS138L, U29 SGP30, U3 Conn_01x04, U30 BSS138L, U31 BSS138L, U32 Micro_SD_Card_Det1, U33 NCV8170AXV300T2G, U4 STM32U595RITx, U5 E22-900M22S, U6 LSM303AH, U7 BME280, U8 ATECC608A-SSHDA, U9 MCP73831-2-OT, X1 SMD3225-4, X2 SMD2012-2

Commit message: pcb: via stitching
Routing:
- net GND: vias 145 -> 267
Other:
- board text added: "PA5"
- board text added: "PC2"

Commit message: pcb: some fixes
Parts:
- moved C40 0.08 mm to (57.7, 89.9)
- moved C41 0.08 mm to (58.7, 89.9)
- moved R50 0.08 mm to (60.1, 90.1)
- moved R51 0.08 mm to (61.2, 90.1)
- moved R15 0.05 mm to (75.5, 31.1)
Routing:
- net (no net): track 4508.9 -> 0.00 mm, vias 705 -> 0
- net GND: track 1183.5 -> 1368.3 mm, vias 267 -> 312
- net I2C1_SCL: track 200.0 -> 198.2 mm
- net HALL_On_Off: track 83.3 -> 82.2 mm
- net VDD_1V8: track 109.4 -> 108.5 mm
- net Net-(U2-RXD1): track 39.0 -> 38.2 mm
- net V_PERIPH_3V: track 316.6 -> 315.9 mm
Other:
- board size 156.3 x 77.5 mm -> 73 x 77.5 mm
