File: uca-dkaiot2-kicad.kicad_pcb (KiCad board)
At the start: 4 copper layers, 73 x 73 mm, 195 parts, among them J1 Conn_01x04, J19 Conn_01x02, J20 Conn_01x01, J21 Conn_01x01, J22 Conn_01x01, J23 Conn_01x01, J27 Conn_01x02, J5 Conn_01x02, J6 Conn_Coaxial, J7 Conn_01x05, J8 USB_B_Micro, Q1 AO3401A, Q2 AO3401A, Q3 AO3400A, Q4 AO3400A, Q5 AO3400A, Q6 AO3400A, SW1 SW_Reed, U1 RT9080-30GJ5, U10 RT9080-30GJ5, U2 Quectel_L96, U23 SPA06-003, U25 FHTC3, U26 OPA2391DGKR, U27 INA3221, U32 Micro_SD_Card_Det1, U33 RT9080-30GJ5, U34 CN3801, U35 TLV320ADC3101, U36 ISL21080CIH315Z-TK, U37 RT9080-30GJ5, U38 OPA379AIDCK, U4 STM32U595RITx, U41 TLV7031DCK, U42 H2112-CB, U43 TMP390, U44 TMP390, U45 LSM6DS3TR-C, U46 RT9080-30GJ5, U47 RT9080-18GJ5, U5 E22-900M22S, X1 SMD3225-4, X2 SMD3215-2 32.768kHz

Commit message: WIP: start routing
Parts:
- removed J5: Conn_01x02, Connector_JST:JST_XH_B2B-XH-A_1x02_P2.50mm_Vertical
- added J2: Conn_01x02, Connector_JST:JST_XH_B2B-XH-A_1x02_P2.50mm_Vertical, F.Cu at (134.4, 78.1)
- added NT1: NetTie_2, NetTie:NetTie-2_SMD_Pad0.5mm, F.Cu at (141.5, 104.5)
- added NT2: NetTie_2, NetTie:NetTie-2_SMD_Pad0.5mm, F.Cu at (182.7, 106.2)
- moved SYM1 59.7 mm to (162.9, 27.8)
- moved C57 5.05 mm to (161.4, 73.2), turned to 90 degrees
- moved R105 4.81 mm to (165.8, 79.5)
- moved R102 4.79 mm to (170.6, 79.5)
- moved R40 2.89 mm to (155.7, 78.4), turned to -90 degrees
- moved C62 1.06 mm to (186.9, 78.3)
- moved C63 1.06 mm to (185.9, 78.3)
- moved R37 0.99 mm to (155.7, 76.4)
- moved C119 0.94 mm to (166.7, 72.0)
- moved R107 0.66 mm to (191.2, 108.2)
- moved U33 0.46 mm to (162.9, 76.0)
- moved C54 0.46 mm to (162.9, 73.7)
- moved C55 0.46 mm to (162.9, 72.7)
- moved C64 0.40 mm to (170.5, 109.2), turned to 180 degrees
- moved U34 0.34 mm to (170.6, 106.0)
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Connections:
- C1 pad 2: -BATT_PROT -> GND
- C10 pad 2: -BATT_PROT -> GND
- C101 pad 2: -BATT_PROT -> GND
- C104 pad 2: -BATT_PROT -> GND
- C106 pad 1: -BATT_PROT -> GND
- C107 pad 2: -BATT_PROT -> GND
- C108 pad 1: -BATT_PROT -> GND
- C109 pad 1: -BATT_PROT -> GND
- C11 pad 2: -BATT_PROT -> GND
- C110 pad 1: +BATT_PROT -> CSON
- C110 pad 2: -BATT_PROT -> GND
- C111 pad 2: -BATT_PROT -> GND
- C115 pad 2: -BATT_PROT -> GND
- C116 pad 2: -BATT_PROT -> GND
- C117 pad 2: -BATT_PROT -> GND
- C119 pad 2: -BATT_PROT -> GND
- C12 pad 2: -BATT_PROT -> GND
- C120 pad 1: +BATT_PROT -> CSON
- C120 pad 2: -BATT_PROT -> GND
- C121 pad 1: +BATT_PROT -> CSON
- C121 pad 2: -BATT_PROT -> GND
- C13 pad 2: -BATT_PROT -> GND
- C14 pad 2: -BATT_PROT -> GND
- C15 pad 2: -BATT_PROT -> GND
- C18 pad 2: -BATT_PROT -> GND
- C19 pad 2: -BATT_PROT -> GND
- C2 pad 2: -BATT_PROT -> GND
- C20 pad 2: -BATT_PROT -> GND
- C28 pad 1: +BATT_PROT -> CSON
- C28 pad 2: -BATT_PROT -> GND
- C29 pad 2: -BATT_PROT -> GND
- C3 pad 2: -BATT_PROT -> GND
- C30 pad 2: -BATT_PROT -> GND
- C4 pad 2: -BATT_PROT -> GND
- C43 pad 2: -BATT_PROT -> GND
- C44 pad 2: -BATT_PROT -> GND
- C45 pad 2: -BATT_PROT -> GND
- C5 pad 2: -BATT_PROT -> GND
- C51 pad 1: +BATT_PROT -> CSON
- C51 pad 2: -BATT_PROT -> GND
- C54 pad 2: -BATT_PROT -> GND
- C55 pad 2: -BATT_PROT -> GND
- C57 pad 1: +BATT_PROT -> CSON
- C57 pad 2: -BATT_PROT -> GND
- C58 pad 2: -BATT_PROT -> GND
- C59 pad 2: -BATT_PROT -> GND
- C6 pad 2: -BATT_PROT -> GND
- C60 pad 2: -BATT_PROT -> GND
- C61 pad 2: -BATT_PROT -> GND
- C62 pad 2: -BATT_PROT -> GND
- C63 pad 2: -BATT_PROT -> GND
- C64 pad 2: -BATT_PROT -> GND
- C66 pad 2: -BATT_PROT -> GND
- C68 pad 2: -BATT_PROT -> GND
- C69 pad 2: -BATT_PROT -> GND
- C7 pad 2: -BATT_PROT -> GND
- C70 pad 2: -BATT_PROT -> GND
- C71 pad 2: -BATT_PROT -> GND
- C75 pad 2: -BATT_PROT -> GND
- C76 pad 2: -BATT_PROT -> GND
- C78 pad 2: -BATT_PROT -> GND
- C79 pad 2: -BATT_PROT -> GND
- C8 pad 2: -BATT_PROT -> GND
- C80 pad 2: -BATT_PROT -> GND
- C81 pad 2: -BATT_PROT -> GND
- C9 pad 2: -BATT_PROT -> GND
- C93 pad 2: -BATT_PROT -> GND
- C94 pad 1: +BATT_PROT -> CSON
- C94 pad 2: -BATT_PROT -> GND
- C96 pad 2: -BATT_PROT -> GND
- C98 pad 2: -BATT_PROT -> GND
- C99 pad 2: -BATT_PROT -> GND
- D9 pad 2: -BATT_PROT -> GND
- J1 pad 1: -BATT_PROT -> GND
- J19 pad 2: -BATT_PROT -> GND
- J21 pad 1: -BATT_PROT -> GND
- J22 pad 1: -BATT_PROT -> GND
- J23 pad 1: -BATT_PROT -> GND
- J27 pad 2: -BATT_PROT -> GND
- J6 pad 2: -BATT_PROT -> GND
- J7 pad 1: -BATT_PROT -> GND
- J8 pad 5: -BATT_PROT -> GND
- J8 pad SH: -BATT_PROT -> GND
- R1 pad 2: -BATT_PROT -> GND
- R114 pad 2: -BATT_PROT -> GND
- R40 pad 2: -BATT_PROT -> GND
- R57 pad 2: -BATT_PROT -> GND
- R65 pad 2: -BATT_PROT -> GND
- R7 pad 2: -BATT_PROT -> GND
- R70 pad 2: +BATT_PROT -> CSON
- R8 pad 2: -BATT_PROT -> GND
- R82 pad 2: -BATT_PROT -> GND
- R84 pad 2: -BATT_PROT -> GND
- R86 pad 2: -BATT_PROT -> GND
- R96 pad 2: -BATT_PROT -> GND
- R99 pad 2: -BATT_PROT -> GND
- SW1 pad 1: -BATT_PROT -> GND
- SW_RST1 pad 1: -BATT_PROT -> GND
- SW_User1 pad 2: -BATT_PROT -> GND
- SYM1 pad 1: -BATT_PROT -> GND
- U1 pad 1: +BATT_PROT -> CSON
- U1 pad 2: -BATT_PROT -> GND
- U10 pad 1: +BATT_PROT -> CSON
- U10 pad 2: -BATT_PROT -> GND
- U10 pad 3: +BATT_PROT -> CSON
- U2 pad 10: -BATT_PROT -> GND
- U2 pad 11: -BATT_PROT -> GND
- U2 pad 12: -BATT_PROT -> GND
- U2 pad 13: -BATT_PROT -> GND
- U2 pad 14: -BATT_PROT -> GND
- U2 pad 15: -BATT_PROT -> GND
- U2 pad 18: -BATT_PROT -> GND
- U2 pad 19: -BATT_PROT -> GND
- U2 pad 21: -BATT_PROT -> GND
- U2 pad 22: -BATT_PROT -> GND
- U2 pad 27: -BATT_PROT -> GND
- U2 pad 31: -BATT_PROT -> GND
- U2 pad 4: -BATT_PROT -> GND
- U2 pad 5: -BATT_PROT -> GND
- U23 pad 1: -BATT_PROT -> GND
- U23 pad 7: -BATT_PROT -> GND
- U25 pad 6: -BATT_PROT -> GND
- U25 pad 7: -BATT_PROT -> GND
- U26 pad 4: -BATT_PROT -> GND
- U27 pad 14: +BATT_PROT -> CSON
- U27 pad 17: -BATT_PROT -> GND
- U27 pad 3: -BATT_PROT -> GND
- U32 pad 6: -BATT_PROT -> GND
- U32 pad SH: -BATT_PROT -> GND
- U33 pad 1: +BATT_PROT -> CSON
- U33 pad 2: -BATT_PROT -> GND
- U34 pad 2: -BATT_PROT -> GND
- U34 pad 7: +BATT_PROT -> CSON
- U35 pad 23: -BATT_PROT -> GND
- U35 pad 25: -BATT_PROT -> GND
- U35 pad 9: -BATT_PROT -> GND
- U36 pad 3: -BATT_PROT -> GND
- U37 pad 1: +BATT_PROT -> CSON
- U37 pad 2: -BATT_PROT -> GND
- U38 pad 2: -BATT_PROT -> GND
- U4 pad 12: -BATT_PROT -> GND
- U4 pad 18: -BATT_PROT -> GND
- U4 pad 31: -BATT_PROT -> GND
- U4 pad 47: -BATT_PROT -> GND
- U4 pad 63: -BATT_PROT -> GND
- U41 pad 2: -BATT_PROT -> GND
- U45 pad 2: -BATT_PROT -> GND
- U45 pad 3: -BATT_PROT -> GND
- U45 pad 6: -BATT_PROT -> GND
- U45 pad 7: -BATT_PROT -> GND
- U46 pad 1: +BATT_PROT -> CSON
- U46 pad 2: -BATT_PROT -> GND
- U47 pad 1: +BATT_PROT -> CSON
- U47 pad 2: -BATT_PROT -> GND
- U5 pad 1: -BATT_PROT -> GND
- U5 pad 10: -BATT_PROT -> GND
- U5 pad 11: -BATT_PROT -> GND
- U5 pad 12: -BATT_PROT -> GND
- U5 pad 2: -BATT_PROT -> GND
- U5 pad 20: -BATT_PROT -> GND
- U5 pad 22: -BATT_PROT -> GND
- U5 pad 3: -BATT_PROT -> GND
- U5 pad 4: -BATT_PROT -> GND
- U5 pad 5: -BATT_PROT -> GND
- X1 pad 2: -BATT_PROT -> GND
- X1 pad 4: -BATT_PROT -> GND
Routing:
- net GND: track 0.00 -> 318.5 mm, vias 0 -> 14
- net CSON: track 0.00 -> 173.7 mm, vias 0 -> 12
- net CSIN: track 0.00 -> 101.6 mm, vias 0 -> 6
- net +3V0_PERIPH: track 0.00 -> 101.1 mm
- net +BATT_PROT: track 0.00 -> 98.4 mm, vias 0 -> 4
- net INT_ACC_2: track 0.00 -> 77.6 mm, vias 0 -> 2
- net INT_ACC_1: track 0.00 -> 76.6 mm, vias 0 -> 2
- net CSOP: track 0.00 -> 73.8 mm, vias 0 -> 4
- net -BATT_OC_OD_PROT: track 0.00 -> 61.8 mm, vias 0 -> 4
- net I2C2_SCL: track 0.00 -> 61.2 mm, vias 0 -> 2
- net MISO_E22: track 0.00 -> 60.8 mm, vias 0 -> 3
- net SCK_E22: track 0.00 -> 57.9 mm, vias 0 -> 3
- net I2C2_SDA: track 0.00 -> 57.9 mm, vias 0 -> 2
- net CSIP: track 0.00 -> 57.2 mm, vias 0 -> 2
- net MOSI_E22: track 0.00 -> 56.3 mm, vias 0 -> 3
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- added copper zone on B.Cu, net GND
- added copper zone on F.Cu, net GND
- added copper zone on In1.Cu, net GND
- added copper zone on In2.Cu, net GND
- removed copper zone on B.Cu, net -BATT_PROT
- removed copper zone on F.Cu, net -BATT_PROT
- removed copper zone on In1.Cu, net -BATT_PROT
- removed copper zone on In2.Cu, net -BATT_PROT
