File: MicrophoneADC.kicad_sch (KiCad schematic)
At the start: 46 parts, among them J18 AudioJack3_SwitchTR, J19 Conn_01x02, J27 Conn_01x02, U35 TLV320ADC3101

Commit message: WIP: BOM
Parts:
- C71: value 1uF/6.3V -> 100nF; LCSC C52923 -> C1525
- C75, C76, C80: value 0.1uF -> 100nF
- C79, C91: value 4.7uF/6.3V -> 4.7µF
- C81: value 1uF/6.3V -> 1uF
- J19, J27: footprint Connector_JST:JST_XH_S2B-XH-A-1_1x02_P2.50mm_Horizontal -> Connector_JST:JST_XH_B2B-XH-A_1x02_P2.50mm_Vertical; LCSC C163035 -> C20079
- R74: value 10k -> 4.7k; JLCPCB Part # (none) -> C25900; LCSC C25744 -> C25900

Commit message: WIP: omit some components and perform initial rough placement on PCB
Parts:
- removed C79: 4.7µF, Capacitor_SMD:C_0402_1005Metric, symbol Device:C_Small
- C73, C83, C84, C85, C86, C87, C88, C89, C90, C91, FB1, R75, R87: now not fitted; now left out of the parts list
- C77, C82: now left out of the parts list
- JP6, JP7, JP8, JP9, TP1, TP2, TP3: now not fitted
Connections:
- net GNDA is gone; now on net GND: C75.2, C78.2, C87.2, C88.2, C89.2, C90.2, C91.2, J18.S, J19.2 (Pin_2), J27.2 (Pin_2), JP6.2 (B), JP7.2 (B), JP8.2 (B), JP9.2 (B), MK1.1 (-), U35.25 (PAD), U35.9 (AVSS)
- net +3.3VA: no longer C75.1, C78.1, U35.10 (AVDD)
- new net +3VSBA: C75.1, C78.1, U35.10 (AVDD)
