File: BatteryProtection.kicad_sch (KiCad schematic)
At the start: 25 parts, among them J29 Conn_01x02, Q3 AO3400A, Q4 AO3400A, Q5 AO3400A, Q6 AO3400A, U42 H2112-CB, U43 TMP390, U44 TMP390

Commit message: WIP: BOM
Parts:
- C112, C113, C114: value 100nF -> 100nF/25V
- R109, R110, R113: now not fitted; now left out of the parts list

Commit message: Finish routing + silkscreen placement
Parts:
- BT1: now left out of the parts list
Changed lines of the file:
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@@
 		(body_style 1)
 		(exclude_from_sim no)
-		(in_bom yes)
+		(in_bom no)
 		(on_board yes)
-		(in_pos_files yes)
+		(in_pos_files no)
 		(dnp no)
 		(property "Reference" "BT1"
