File: MicrophoneTrigger.kicad_sch (KiCad schematic)
At the start: 43 parts, among them U36 ISL21080CIH315Z-TK, U37 RT9080-30GJ5, U38 OPA379AIDCK, U39 OPA391DCKR, U40 OPA391DCKR, U41 TLV7031DCK

Commit message: WIP: BOM
Parts:
- removed C110: 0.1µF/6.3V, Capacitor_SMD:C_0402_1005Metric, symbol Device:C_Small
- removed U39, U40: OPA391DCKR, Package_TO_SOT_SMD:SOT-353_SC-70-5, symbol PCM_Amplifier_Operational_AKL:OPA379AIDCK
- added U26: OPA2391DGKR, PCM_Package_SO_AKL:MSOP-8_3x3mm_P0.65mm, symbol PCM_Amplifier_Operational_AKL:OPA2388IDGK
- C101, C96: value 4.7µF/6.3V -> 4.7µF
- C105: value 4.7uF/6.3V -> 4.7µF
- C106, C108, C109: LCSC (none) -> C12530
- C107, C111, C93, C99: value 0.1µF/6.3V -> 100nF
- C95, C97: LCSC (none) -> C15195
- C98: value 10nF/6.3V -> 10nF
- R100, R93, R97: LCSC (none) -> C25900
- R91: LCSC (none) -> C25744
- R94, R96, R99: LCSC (none) -> C25741
- U37: LCSC Part C965900 -> (none)
Connections:
- net +3VSBA: now also U26.8 (V+)
- net GNDA: now also U26.4 (V-)
- net at R89.1, R91.1, U38.3 (-)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: now also U26.3 (+)
- net at R93.1, R94.1: now also U26.2 (-)
- net at R94.2: now also U26.1, U26.5 (+)
- net at D11.2 (A), R95.1, RV4.2: now also U26.7
- net at R100.1, R97.1: now also U26.6 (-)

Commit message: WIP: omit some components and perform initial rough placement on PCB
Parts:
- C104: value 100uF/6.3V -> 47uF/6.3V; LCSC C15008 -> C96123
- C105: now not fitted; now left out of the parts list
- C92: now left out of the parts list
Changed lines of the file:
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@@
 			)
 		)
-		(property "Value" "100uF/6.3V"
+		(property "Value" "47uF/6.3V"
 			(at 111.76 133.604 0)
 			(show_name no)
@@
 			)
 		)
-		(property "LCSC" "C15008"
-			(at 116.84 127 0)
-			(hide yes)
-			(show_name no)
-			(do_not_autoplace no)
-			(effects
-				(font
-					(size 1.27 1.27)
-				)
-			)
-		)
-		(property "LCSC Part" ""
+		(property "LCSC" "C96123"
 			(at 116.84 127 0)
 			(hide yes)
@@
 		(body_style 1)
 		(exclude_from_sim no)
-		(in_bom yes)
-		(on_board yes)
-		(in_pos_files yes)
+		(in_bom no)
+		(on_board no)
+		(in_pos_files no)
 		(dnp yes)
 		(property "Reference" "C92"
@@
 		(body_style 1)
 		(exclude_from_sim no)
-		(in_bom yes)
-		(on_board yes)
-		(in_pos_files yes)
-		(dnp no)
+		(in_bom no)
+		(on_board no)
+		(in_pos_files no)
+		(dnp yes)
 		(property "Reference" "C105"
 			(at 123.698 124.714 0)

Commit message: Finish routing + silkscreen placement
Parts:
- U26: FT Rotation Offset (none) -> -90
Changed lines of the file:
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@@
 			)
 		)
+		(property "FT Rotation Offset" "-90"
+			(at 215.9 40.64 0)
+			(hide yes)
+			(show_name no)
+			(do_not_autoplace no)
+			(effects
+				(font
+					(size 1.27 1.27)
+				)
+			)
+		)
 		(pin "8"
 		)
@@
 			(at 143.51 40.64 0)
 			(hide yes)
+			(show_name no)
+			(do_not_autoplace no)
+			(effects
+				(font
+					(size 1.27 1.27)
+				)
+			)
+		)
+		(property "FT Rotation Offset" "-90"
+			(at 143.51 40.64 0)
+			(hide yes)
