File: Power_Monitor_Charger.kicad_sch (KiCad schematic)
At the start: 57 parts, among them J13 Conn_01x04, J14 Conn_01x04, J15 Conn_01x02, J16 Conn_01x02, J17 Conn_01x02, J2 Conn_01x02, J9 Conn_01x02, Q1 AO3401A, Q2 AO3401A, U27 INA3221, U34 CN3801

Commit message: WIP: BOM
Parts:
- C62: value 4.7µF/6.3V -> 4.7µF
- C63: value 100nF/6.3V -> 100nF
- C67: now not fitted; now left out of the parts list
- J13: footprint Connector_PinHeader_2.54mm:PinHeader_1x04_P2.54mm_Vertical -> Connector_JST:JST_XH_B4B-XH-A_1x04_P2.50mm_Vertical; LCSC (none) -> C37815
- J15, J9: footprint Connector_JST:JST_XH_S2B-XH-A_1x02_P2.50mm_Horizontal -> Connector_JST:JST_XH_B2B-XH-A_1x02_P2.50mm_Vertical; LCSC C157931 -> C20079
- J16, J2: footprint Connector_JST:JST_XH_S2B-XH-A-1_1x02_P2.50mm_Horizontal -> Connector_JST:JST_XH_B2B-XH-A_1x02_P2.50mm_Vertical; LCSC C163035 -> C20079
- J17: footprint Connector_PinSocket_2.54mm:PinSocket_1x02_P2.54mm_Vertical -> Connector_JST:JST_XH_B2B-XH-A_1x02_P2.50mm_Vertical; LCSC C157931 -> C20079; now left out of the parts list
- L1: value 47µH/3A -> 33µH/2.32A; footprint Inductor_SMD:L_Sunlord_MWSA0804S -> Inductor_SMD:L_Chilisin_BMRB00060650; LCSC C2962889 -> C47327223
- Q1, Q2: LCSC (none) -> C15127
- U34: LCSC (none) -> C840499; LCSC Part C840499 -> (none)

Commit message: WIP: start routing
Parts:
- added NT1, NT2, NT3: NetTie_2, NetTie:NetTie-2_SMD_Pad0.5mm, symbol Device:NetTie_2
- J2: now fitted; now in the parts list
Connections:
- net +BATT: now also NT1.1
- net GND: now also NT2.1
- net SOLAR: now also NT3.2; no longer C44.1, C45.1, C60.1, C61.1, D12.1 (K), J2.1 (Pin_1), R32.1, R33.1, U27.12 (IN+1)
- new net +BATT_PROT: NT1.2
- new net -BATT_PROT: NT2.2
- new net CSIP: C44.1, C45.1, C60.1, C61.1, D12.1 (K), J2.1 (Pin_1), NT3.1, R32.1, R33.1, U27.12 (IN+1)
